File: LorisBurnWire.sch (KiCad schematic (older format))
At the start: 54 parts, among them J1 BurnWire, J2 BurnWire, J3 BurnWire, J4 BurnWire, Q1 BUK7M6R3-40EX, Q2 BUK7M6R3-40EX, Q3 BUK7M6R3-40EX, Q4 BUK7M6R3-40EX, U1 TLC555ID, U2 TLC555ID, U3 LP38501-ADJ, U4 TLC555ID, U5 LMP8646, U6 TLC555ID

Commit message: Fixed footprint applied to burnwire
Parts:
- J1, J2, J3, J4: footprint TerminalBlock_Phoenix:TerminalBlock_Phoenix_MKDS-3-2-5.08_1x02_P5.08mm_Horizontal -> TempoFootprints:TE_282837-2
Changed lines of the file:
@@
 F 0 "J4" H 9405 8167 50  0000 L CNN
 F 1 "BurnWire" H 9405 8076 50  0000 L CNN
-F 2 "TerminalBlock_Phoenix:TerminalBlock_Phoenix_MKDS-3-2-5.08_1x02_P5.08mm_Horizontal" H 9325 8175 50  0001 C CNN
+F 2 "TempoFootprints:TE_282837-2" H 9325 8175 50  0001 C CNN
 F 3 "~" H 9325 8175 50  0001 C CNN
 	1    9325 8175
@@
 F 0 "J3" H 7055 8167 50  0000 L CNN
 F 1 "BurnWire" H 7055 8076 50  0000 L CNN
-F 2 "TerminalBlock_Phoenix:TerminalBlock_Phoenix_MKDS-3-2-5.08_1x02_P5.08mm_Horizontal" H 6975 8175 50  0001 C CNN
+F 2 "TempoFootprints:TE_282837-2" H 6975 8175 50  0001 C CNN
 F 3 "~" H 6975 8175 50  0001 C CNN
 	1    6975 8175
@@
 F 0 "J2" H 4980 8167 50  0000 L CNN
 F 1 "BurnWire" H 4980 8076 50  0000 L CNN
-F 2 "TerminalBlock_Phoenix:TerminalBlock_Phoenix_MKDS-3-2-5.08_1x02_P5.08mm_Horizontal" H 4900 8175 50  0001 C CNN
+F 2 "TempoFootprints:TE_282837-2" H 4900 8175 50  0001 C CNN
 F 3 "~" H 4900 8175 50  0001 C CNN
 	1    4900 8175
@@
 F 0 "J1" H 2630 8142 50  0000 L CNN
 F 1 "BurnWire" H 2630 8051 50  0000 L CNN
-F 2 "TerminalBlock_Phoenix:TerminalBlock_Phoenix_MKDS-3-2-5.08_1x02_P5.08mm_Horizontal" H 2550 8150 50  0001 C CNN
+F 2 "TempoFootprints:TE_282837-2" H 2550 8150 50  0001 C CNN
 F 3 "~" H 2550 8150 50  0001 C CNN
 	1    2550 8150

Commit message: updated jumper wire footprint
Parts:
- JP1: footprint (none) -> TempoFootprints:TE_87224-3
Changed lines of the file:
@@
 F 0 "JP1" H 5600 2000 50  0000 C CNN
 F 1 "Jumper_3_Open" H 5675 2075 50  0000 C CNN
-F 2 "" H 5350 1875 50  0001 C CNN
+F 2 "TempoFootprints:TE_87224-3" H 5350 1875 50  0001 C CNN
 F 3 "~" H 5350 1875 50  0001 C CNN
 	1    5350 1875
